File: HeisserDraht/HeisserDraht.kicad_pcb (KiCad board)
At the start: 2 copper layers, 29.6 x 85 mm, 18 parts, among them J1 Pen, J2 Track, Q1 BC547, Q2 BC547, Q3 BC547, SW2 SW_DPST_x2, SW3 SW_SPDT_321

Commit message: updated resistore values
Parts:
- R1, R3: value R -> 470
- R2, R4: value R -> 47k
- R5, R6: value R -> 1k
- R7: value R -> 100k
Changed lines of the file:
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@@
 			)
 		)
-		(property "Value" "R"
+		(property "Value" "47k"
 			(at 5.08 2.54 90)
 			(layer "F.Fab")
@@
 			)
 		)
-		(property "Value" "R"
+		(property "Value" "1k"
 			(at 5.08 2.37 180)
 			(layer "F.Fab")
@@
 			)
 		)
-		(property "Value" "R"
+		(property "Value" "1k"
 			(at 5.08 2.37 180)
 			(layer "F.Fab")
@@
 			)
 		)
-		(property "Value" "R"
+		(property "Value" "47k"
 			(at 5.08 2.37 90)
 			(layer "F.Fab")
@@
 			)
 		)
-		(property "Value" "R"
+		(property "Value" "470"
 			(at 5.08 2.37 -90)
 			(layer "F.Fab")
@@
 			)
 		)
-		(property "Value" "R"
+		(property "Value" "100k"
 			(at 5.08 2.37 90)
 			(layer "F.Fab")
@@
 			)
 		)
-		(property "Value" "R"
+		(property "Value" "470"
 			(at 5.08 2.37 90)
 			(layer "F.Fab")
