File: HeisserDraht/HeisserDraht.kicad_sch (KiCad schematic)
At the start: 18 parts, among them J1 Pen, J2 Track, Q1 BC547, Q2 BC547, Q3 BC547, SW2 SW_DPST_x2, SW3 SW_SPDT_321

Commit message: updated resistore values
Parts:
- R1, R3: value R -> 470
- R2, R4: value R -> 47k
- R5, R6: value R -> 1k
- R7: value R -> 100k
Changed lines of the file:
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@@
 			)
 		)
-		(property "Value" "R"
+		(property "Value" "470"
 			(at 142.24 82.5499 0)
 			(effects
@@
 			)
 		)
-		(property "Value" "R"
+		(property "Value" "47k"
 			(at 153.67 95.553 90)
 			(effects
@@
 			)
 		)
-		(property "Value" "R"
+		(property "Value" "100k"
 			(at 115.57 59.69 90)
 			(effects
@@
 			)
 		)
-		(property "Value" "R"
+		(property "Value" "47k"
 			(at 179.07 95.25 90)
 			(effects
@@
 			)
 		)
-		(property "Value" "R"
+		(property "Value" "1k"
 			(at 130.81 95.2499 0)
 			(effects
@@
 			)
 		)
-		(property "Value" "R"
+		(property "Value" "470"
 			(at 189.23 82.5499 0)
 			(effects
@@
 			)
 		)
-		(property "Value" "R"
+		(property "Value" "1k"
 			(at 204.47 95.2499 0)
 			(effects
